File: schematics/schematics.sch (KiCad schematic (older format))
At the start: 8 parts, among them J1 Conn_01x06_Female, J2 Conn_01x07_Female, U1 ATmega8A-PU, U2 AMS1117-3.3, U3 NRF24L01_Breakout

Commit message: Schematics are done
Parts:
- removed J1: Conn_01x06_Female, symbol Connector:Conn_01x06_Female
- added J1: Conn_01x02, Connector_Wire:SolderWirePad_1x02_P3.81mm_Drill0.8mm, symbol Connector_Generic:Conn_01x02
- J2: footprint (none) -> Connector_PinHeader_2.54mm:PinHeader_1x07_P2.54mm_Vertical
- R1, R2, R3: footprint (none) -> Resistor_THT:R_Axial_DIN0204_L3.6mm_D1.6mm_P5.08mm_Horizontal
Connections:
- net BATTERY_IN: now also J1.1 (Pin_1)
- net GND: now also U2.1 (GND), J1.2 (Pin_2)
- net AVR_RX: now reaches U1.2 (PD0)
- net AVR_TX: now reaches U1.3 (PD1)
- no-connect marks 1 -> 0
Changed lines of the file:
@@
 F 0 "R2" H 6600 1050 50  0000 L CNN
 F 1 "220k" H 6600 950 50  0000 L CNN
-F 2 "" V 6430 1050 50  0001 C CNN
+F 2 "Resistor_THT:R_Axial_DIN0204_L3.6mm_D1.6mm_P5.08mm_Horizontal" V 6430 1050 50  0001 C CNN
 F 3 "~" H 6500 1050 50  0001 C CNN
 	1    6500 1050
@@
 F 0 "R3" H 6600 1350 50  0000 L CNN
 F 1 "220k" H 6600 1250 50  0000 L CNN
-F 2 "" V 6430 1350 50  0001 C CNN
+F 2 "Resistor_THT:R_Axial_DIN0204_L3.6mm_D1.6mm_P5.08mm_Horizontal" V 6430 1350 50  0001 C CNN
 F 3 "~" H 6500 1350 50  0001 C CNN
 	1    6500 1350
@@
 F 0 "R1" H 3600 2150 50  0000 L CNN
 F 1 "220k" H 3600 2050 50  0000 L CNN
-F 2 "" V 3780 2050 50  0001 C CNN
+F 2 "Resistor_THT:R_Axial_DIN0204_L3.6mm_D1.6mm_P5.08mm_Horizontal" V 3780 2050 50  0001 C CNN
 F 3 "~" H 3850 2050 50  0001 C CNN
 	1    3850 2050
@@
 F 0 "J2" H 7178 3726 50  0000 L CNN
 F 1 "Conn_01x07_Female" H 7178 3635 50  0000 L CNN
-F 2 "" H 7150 3700 50  0001 C CNN
+F 2 "Connector_PinHeader_2.54mm:PinHeader_1x07_P2.54mm_Vertical" H 7150 3700 50  0001 C CNN
 F 3 "~" H 7150 3700 50  0001 C CNN
 	1    7150 3700
@@
 Text Label 4550 1900 1    50   ~ 0
 BATTERY_IN
+Text Label 3850 2200 2    50   ~ 0
+AVR_RST
+Text Label 8200 1300 3    50   ~ 0
+GND
+Text Label 5050 3600 0    50   ~ 0
+AVR_RX
+Text Label 5050 3700 0    50   ~ 0
+AVR_TX
 $Comp
-L Connector:Conn_01x06_Female J1
-U 1 1 5E4559E2
-P 6200 4800
-F 0 "J1" H 6228 4776 50  0000 L CNN
-F 1 "Conn_01x06_Female" H 6228 4685 50  0000 L CNN
-F 2 "" H 6200 4800 50  0001 C CNN
-F 3 "~" H 6200 4800 50  0001 C CNN
-	1    6200 4800
+L Connector_Generic:Conn_01x02 J1
+U 1 1 5E43D109
+P 5850 4300
+F 0 "J1" H 5930 4292 50  0000 L CNN
+F 1 "Conn_01x02" H 5930 4201 50  0000 L CNN
+F 2 "Connector_Wire:SolderWirePad_1x02_P3.81mm_Drill0.8mm" H 5850 4300 50  0001 C CNN
+F 3 "~" H 5850 4300 50  0001 C CNN
+	1    5850 4300
 	1    0    0    -1
 $EndComp
-Text Label 6000 4600 2    50   ~ 0
+Text Label 5650 4400 3    50   ~ 0
 GND
-NoConn ~ 6000 4700
-Text Label 3850 2200 2    50   ~ 0
-AVR_RST
-Text Label 6000 4800 2    50   ~ 0
-AVR_RST
-Text Label 6000 4900 2    50   ~ 0
-NRF_SCK
-Text Label 6000 5000 2    50   ~ 0
-NRF_MISO
-Text Label 6000 5100 2    50   ~ 0
-NRF_MOSI
+Text Label 5650 4300 2    50   ~ 0
+BATTERY_IN
 $EndSCHEMATC

Commit message: Updated PCB.
Parts:
- removed R2, R3: 220k, Resistor_THT:R_Axial_DIN0204_L3.6mm_D1.6mm_P5.08mm_Horizontal, symbol Device:R
- J1: value Conn_01x02 -> POWER; footprint Connector_Wire:SolderWirePad_1x02_P3.81mm_Drill0.8mm -> Connector_PinHeader_2.00mm:PinHeader_1x02_P2.00mm_Vertical
- J2: value Conn_01x07_Female -> PSX_CONNECTOR
- U3: value NRF24L01_Breakout -> NRF24L01_BREAKOUT
Connections:
- net ADC_IN: no longer names the net of U1.23 (PC0)
Changed lines of the file:
@@
 	1    0    0    -1
 $EndComp
-$Comp
-L Device:R R2
-U 1 1 5E43C370
-P 6500 1050
-F 0 "R2" H 6600 1050 50  0000 L CNN
-F 1 "220k" H 6600 950 50  0000 L CNN
-F 2 "Resistor_THT:R_Axial_DIN0204_L3.6mm_D1.6mm_P5.08mm_Horizontal" V 6430 1050 50  0001 C CNN
-F 3 "~" H 6500 1050 50  0001 C CNN
-	1    6500 1050
-	1    0    0    -1
-$EndComp
-$Comp
-L Device:R R3
-U 1 1 5E43D361
-P 6500 1350
-F 0 "R3" H 6600 1350 50  0000 L CNN
-F 1 "220k" H 6600 1250 50  0000 L CNN
-F 2 "Resistor_THT:R_Axial_DIN0204_L3.6mm_D1.6mm_P5.08mm_Horizontal" V 6430 1350 50  0001 C CNN
-F 3 "~" H 6500 1350 50  0001 C CNN
-	1    6500 1350
-	1    0    0    -1
-$EndComp
-Text Label 6500 1200 2    50   ~ 0
-ADC_IN
-Text Label 5050 2900 0    50   ~ 0
-ADC_IN
-Text Label 6500 900  0    50   ~ 0
-BATTERY_IN
-Text Label 6500 1500 3    50   ~ 0
-GND
 Text Label 4550 4700 3    50   ~ 0
 GND
@@
 P 7150 3700
 F 0 "J2" H 7178 3726 50  0000 L CNN
-F 1 "Conn_01x07_Female" H 7178 3635 50  0000 L CNN
+F 1 "PSX_CONNECTOR" H 7178 3635 50  0000 L CNN
 F 2 "Connector_PinHeader_2.54mm:PinHeader_1x07_P2.54mm_Vertical" H 7150 3700 50  0001 C CNN
 F 3 "~" H 7150 3700 50  0001 C CNN
@@
 P 8750 2700
 F 0 "U3" H 9130 2746 50  0000 L CNN
-F 1 "NRF24L01_Breakout" H 9130 2655 50  0000 L CNN
+F 1 "NRF24L01_BREAKOUT" H 9130 2655 50  0000 L CNN
 F 2 "RF_Module:nRF24L01_Breakout" H 8900 3300 50  0001 L CIN
 F 3 "http://www.nordicsemi.com/eng/content/download/2730/34105/file/nRF24L01_Product_Specification_v2_0.pdf" H 8750 2600 50  0001 C CNN
@@
 P 5850 4300
 F 0 "J1" H 5930 4292 50  0000 L CNN
-F 1 "Conn_01x02" H 5930 4201 50  0000 L CNN
-F 2 "Connector_Wire:SolderWirePad_1x02_P3.81mm_Drill0.8mm" H 5850 4300 50  0001 C CNN
+F 1 "POWER" H 5930 4201 50  0000 L CNN
+F 2 "Connector_PinHeader_2.00mm:PinHeader_1x02_P2.00mm_Vertical" H 5850 4300 50  0001 C CNN
 F 3 "~" H 5850 4300 50  0001 C CNN
 	1    5850 4300
